File: calypso.kicad_pcb (KiCad board)
At the start: 2 copper layers, 99.1 x 99.1 mm, 91 parts, among them IC1 RP2040_breakout, J1 Conn_01x06, J10 AudioJack3, J11 AudioJack3, J13 Joy, J14 Video Out, J15 DB15_Female_HighDensity, J2 Conn_02x12_Odd_Even, J3 Mini-DIN-6, J4 Mini-DIN-6, J5 Conn_01x05, J6 Micro_SD_Card, J7 USB_B_Mini, Q1 BC846, Q2 BC846, SW1 SWDPDTBLUE, SW2 SW_Push, U1 AMS1117-3.3, U2 PCM5102, U3 CYC1000

Commit message: test
Parts:
- C11, C12, C13, C15, C16, C17, C3, C5, C6, C8, C9: footprint Capacitor_SMD:C_1206_3216Metric_Pad1.33x1.80mm_HandSolder -> Capacitor_SMD:C_0805_2012Metric_Pad1.18x1.45mm_HandSolder
- C7: footprint Capacitor_SMD:C_1206_3216Metric_Pad1.33x1.80mm_HandSolder -> Capacitor_Tantalum_SMD:CP_EIA-3216-12_Kemet-S_Pad1.58x1.35mm_HandSolder
- D1: footprint Diode_SMD:D_MiniMELF -> Diode_SMD:D_SOD-123F
- D13: footprint LED_SMD:LED_1206_3216Metric_Pad1.42x1.75mm_HandSolder -> LED_SMD:LED_0805_2012Metric_Pad1.15x1.40mm_HandSolder
- R1, R10, R11, R12, R13, R16, R17, R18, R19, R20, R21, R22, R24, R25, R26, R27, R28, R29, R3, R30, R31, R32, R33, R34, R35, R36, R37, R38, R39, R4, R40, R41, R42, R43, R44, R45, R5, R6, R7, R8, R9: footprint Resistor_SMD:R_1206_3216Metric_Pad1.30x1.75mm_HandSolder -> Resistor_SMD:R_0805_2012Metric_Pad1.20x1.40mm_HandSolder
- moved R20 15.2 mm to (51.8, 41.4), turned to 180 degrees
- moved R16 11.4 mm to (62.2, 44.7), turned to 180 degrees
- moved R19 10.7 mm to (51.8, 44.7), turned to 180 degrees
- moved R44 9.03 mm to (65.9, 86.9)
- moved C17 8.41 mm to (104.9, 45.5), turned to 0 degrees
- moved R17 7.35 mm to (62.2, 47.8), turned to 180 degrees
- moved C16 6.18 mm to (104.9, 52.6), turned to 0 degrees
- moved R26 5.41 mm to (65.5, 32.8), turned to 180 degrees
- moved R18 4.58 mm to (62.2, 50.5), turned to 180 degrees
- moved R33 4.32 mm to (37.7, 46.0)
- moved R34 4.32 mm to (37.8, 41.7)
- moved R3 4.08 mm to (118.6, 38.7)
- moved R1 3.33 mm to (115.3, 38.7)
- moved D13 2.79 mm to (81.8, 85.3), turned to 0 degrees
- moved R45 1.78 mm to (88.1, 85.3), turned to 180 degrees
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Routing:
- net GND: track 919.2 -> 851.1 mm, vias 1 -> 34
- net RP_GP29: track 47.7 -> 27.3 mm
- net Net-(C16-Pad1): track 36.4 -> 17.9 mm
- net C10_J1: track 45.8 -> 63.5 mm
- net C10_P2: track 57.9 -> 41.2 mm
- net +5V: track 309.7 -> 320.7 mm
- net C10_P1: track 62.5 -> 52.9 mm
- net C10_J2: track 65.8 -> 56.3 mm
- net JOY_RIGHT: track 57.3 -> 65.1 mm, vias 1 -> 2
- net Net-(J14-Pad2): track 12.9 -> 5.39 mm
- net Net-(C17-Pad1): track 28.3 -> 21.0 mm
- net Net-(C9-Pad2): track 11.6 -> 4.92 mm
- net C10_R11: track 104.0 -> 97.5 mm
- net +3.3VP: track 383.9 -> 389.9 mm
- net Net-(J10-PadR): track 43.6 -> 38.3 mm
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Other:
- board text added: "JLCJLCJLCJLC"
