File: power.kicad_sch (KiCad schematic)
At the start: 9 parts, among them J7 USB_B_Mini, SW1 SWDPDTBLUE, SW2 SW_Push, U1 AMS1117-3.3

Commit message: test
Parts:
- C1, C2: LCSC (none) -> C7171
- C3: footprint Capacitor_SMD:C_1206_3216Metric_Pad1.33x1.80mm_HandSolder -> Capacitor_SMD:C_0805_2012Metric_Pad1.18x1.45mm_HandSolder; LCSC (none) -> C28233
- D13: footprint LED_SMD:LED_1206_3216Metric_Pad1.42x1.75mm_HandSolder -> LED_SMD:LED_0805_2012Metric_Pad1.15x1.40mm_HandSolder; LCSC (none) -> C2297
- J7: LCSC (none) -> C3039330
- R45: footprint Resistor_SMD:R_1206_3216Metric_Pad1.30x1.75mm_HandSolder -> Resistor_SMD:R_0805_2012Metric_Pad1.20x1.40mm_HandSolder; LCSC (none) -> C17513
- U1: LCSC (none) -> C6186
